File: voltage_sense.kicad_pcb (KiCad board)
At the start: 6 copper layers, 48 x 34 mm, 95 parts, among them IC1 DAC101C081CIMK_NOPB, J1 Conn_Coaxial, J2 DNI, J4 HDMI_A, J5 Conn_Coaxial, U1 OPA188xxDBV, U10 TMUX6111PWR, U11 REF3440TIDBVR, U2 TCA9555DBR, U3 OPA188xxDBV, U4 MCP4017T-103E_LT, U5 OPA1641, U6 24AA025UID, U7 ADA4000-2ARZ-R7, U8 TMUX6111PWR, U9 LP2981A-33DBVT

Commit message: All production files in jlcpcb/production_files
Changed lines of the file:
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@@
     (descr "http://www.farnell.com/datasheets/612848.pdf")
     (tags "BNC Amphenol Horizontal")
-    (property "Manf#" "C2874827")
     (property "Sheetfile" "voltage_sense_top.kicad_sch")
     (property "Sheetname" "vsense")
@@
     (fp_arc (start 5.5 -3) (mid 5.353553 -2.646447) (end 5 -2.5) (layer "F.SilkS") (width 0.127))
     (fp_arc (start 4.5 -2.5) (mid 4.146447 -2.646447) (end 4 -3) (layer "F.SilkS") (width 0.127))
-    (fp_arc (start 5.075468 -0.778281) (mid 5.142434 -0.901086) (end 5.273459 -0.949998) (layer "F.SilkS") (width 0.127))
+    (fp_arc (start 5.075468 -0.778281) (mid 5.142414 -0.901105) (end 5.273459 -0.949998) (layer "F.SilkS") (width 0.127))
     (fp_arc (start -5.4719 -0.7752) (mid -5.423377 -0.932365) (end -5.273441 -1.000001) (layer "F.SilkS") (width 0.127))
     (fp_arc (start -3.25 3.75) (mid -3.396447 4.103553) (end -3.75 4.25) (layer "F.SilkS") (width 0.127))
     (fp_arc (start -5 -2.5) (mid -5.353553 -2.646447) (end -5.5 -3) (layer "F.SilkS") (width 0.127))
     (fp_arc (start -2 -3.7) (mid -2.058579 -3.558579) (end -2.2 -3.5) (layer "F.SilkS") (width 0.127))
-    (fp_arc (start 5.373443 -0.95) (mid 5.523389 -0.882352) (end 5.571899 -0.725198) (layer "F.SilkS") (width 0.127))
+    (fp_arc (start 5.373443 -0.95) (mid 5.523346 -0.882348) (end 5.571899 -0.725198) (layer "F.SilkS") (width 0.127))
     (fp_arc (start 2.2 -3.5) (mid 2.058579 -3.558579) (end 2 -3.7) (layer "F.SilkS") (width 0.127))
-    (fp_arc (start 3.42654 -0.95) (mid 3.557588 -0.901082) (end 3.62453 -0.778279) (layer "F.SilkS") (width 0.127))
+    (fp_arc (start 3.42654 -0.95) (mid 3.55756 -0.901074) (end 3.62453 -0.778279) (layer "F.SilkS") (width 0.127))
     (fp_arc (start 5.35 3.8) (mid 5.203553 4.153553) (end 4.85 4.3) (layer "F.SilkS") (width 0.127))
     (fp_arc (start -2.3 -3.5) (mid -2.441421 -3.558579) (end -2.5 -3.7) (layer "F.SilkS") (width 0.127))
@@
     (fp_line (start -1.113417 1.125451) (end -1.081286 1.125451) (layer "B.Fab") (width 0.127))
     (fp_line (start 1.421808 0.750547) (end 1.421808 1.125451) (layer "B.Fab") (width 0.127))
-    (fp_arc (start -0.576537 0.906071) (mid -0.449563 0.779101) (end -0.322588 0.906071) (layer "B.Fab") (width 0.127))
+    (fp_arc (start -0.576537 0.906071) (mid -0.449563 0.779106) (end -0.322588 0.906071) (layer "B.Fab") (width 0.127))
     (fp_arc (start -0.724999 1.446) (mid -0.778512 1.423533) (end -0.800692 1.369901) (layer "B.Fab") (width 0.127))
     (fp_arc (start -0.800692 -1.398928) (mid -0.778507 -1.452548) (end -0.724999 -1.475002) (layer "B.Fab") (width 0.127))
@@
     (connect_pads (clearance 0))
     (min_thickness 0.254)
-    (keepout (tracks allowed) (vias allowed) (pads allowed) (copperpour not_allowed) (footprints allowed))
+    (keepout (tracks allowed) (vias allowed) (pads allowed ) (copperpour not_allowed) (footprints allowed))
     (fill (thermal_gap 0.508) (thermal_bridge_width 0.508))
     (polygon
@@
     (connect_pads (clearance 0))
     (min_thickness 0.254)
-    (keepout (tracks allowed) (vias allowed) (pads allowed) (copperpour not_allowed) (footprints allowed))
+    (keepout (tracks allowed) (vias allowed) (pads allowed ) (copperpour not_allowed) (footprints allowed))
     (fill (thermal_gap 0.508) (thermal_bridge_width 0.508))
     (polygon

Commit message: add modified production files; schematic update by KiCAD version to 8.0.1
Parts:
- moved R34 0.25 mm to (26.8, -17.9)
Changed lines of the file:
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@@
     (property "Sheetname" "vsense")
     (attr smd)
-    (fp_text reference "U7" (at 0 0 90 unlocked) (layer "F.SilkS")
+    (fp_text reference "U7" (at 2.2733 -3.4417 90 unlocked) (layer "F.SilkS")
       (effects (font (size 1 1) (thickness 0.15)))
     )
@@
     (property "Sheetname" "vsense")
     (attr through_hole)
-    (fp_text reference "J2" (at 4.385 -2.27 90) (layer "F.SilkS")
+    (fp_text reference "J2" (at -0.324 -2.55 90) (layer "F.SilkS")
       (effects (font (size 1 1) (thickness 0.15)))
     )
@@
     (property "Tolerance" "1%")
     (attr smd)
-    (fp_text reference "R13" (at -0.127 -1.397 90) (layer "F.SilkS")
+    (fp_text reference "R13" (at 0.762 1.524 90) (layer "F.SilkS")
       (effects (font (size 1 1) (thickness 0.15)))
     )
@@
     (property "Status" "Active")
     (attr smd)
-    (fp_text reference "U4" (at 2.413 -1.016) (layer "F.SilkS")
+    (fp_text reference "U4" (at 0.127 -2.286) (layer "F.SilkS")
       (effects (font (size 1 1) (thickness 0.15)))
     )
@@
     (property "Tolerance" "1%")
     (attr smd)
-    (fp_text reference "R26" (at -2.159 0.508) (layer "F.SilkS")
+    (fp_text reference "R26" (at -0.254 1.397 90) (layer "F.SilkS")
       (effects (font (size 1 1) (thickness 0.15)))
     )
@@
     (fp_arc (start 5.5 -3) (mid 5.353553 -2.646447) (end 5 -2.5) (layer "F.SilkS") (width 0.127))
     (fp_arc (start 4.5 -2.5) (mid 4.146447 -2.646447) (end 4 -3) (layer "F.SilkS") (width 0.127))
-    (fp_arc (start 5.075468 -0.778281) (mid 5.142414 -0.901105) (end 5.273459 -0.949998) (layer "F.SilkS") (width 0.127))
+    (fp_arc (start 5.075468 -0.778281) (mid 5.142422 -0.901068) (end 5.273459 -0.949998) (layer "F.SilkS") (width 0.127))
     (fp_arc (start -5.4719 -0.7752) (mid -5.423377 -0.932365) (end -5.273441 -1.000001) (layer "F.SilkS") (width 0.127))
     (fp_arc (start -3.25 3.75) (mid -3.396447 4.103553) (end -3.75 4.25) (layer "F.SilkS") (width 0.127))
     (fp_arc (start -5 -2.5) (mid -5.353553 -2.646447) (end -5.5 -3) (layer "F.SilkS") (width 0.127))
     (fp_arc (start -2 -3.7) (mid -2.058579 -3.558579) (end -2.2 -3.5) (layer "F.SilkS") (width 0.127))
-    (fp_arc (start 5.373443 -0.95) (mid 5.523346 -0.882348) (end 5.571899 -0.725198) (layer "F.SilkS") (width 0.127))
+    (fp_arc (start 5.373443 -0.95) (mid 5.523389 -0.882352) (end 5.571899 -0.725198) (layer "F.SilkS") (width 0.127))
     (fp_arc (start 2.2 -3.5) (mid 2.058579 -3.558579) (end 2 -3.7) (layer "F.SilkS") (width 0.127))
-    (fp_arc (start 3.42654 -0.95) (mid 3.55756 -0.901074) (end 3.62453 -0.778279) (layer "F.SilkS") (width 0.127))
+    (fp_arc (start 3.42654 -0.95) (mid 3.557588 -0.901082) (end 3.62453 -0.778279) (layer "F.SilkS") (width 0.127))
     (fp_arc (start 5.35 3.8) (mid 5.203553 4.153553) (end 4.85 4.3) (layer "F.SilkS") (width 0.127))
     (fp_arc (start -2.3 -3.5) (mid -2.441421 -3.558579) (end -2.5 -3.7) (layer "F.SilkS") (width 0.127))
@@
     (fp_line (start -1.113417 1.125451) (end -1.081286 1.125451) (layer "B.Fab") (width 0.127))
     (fp_line (start 1.421808 0.750547) (end 1.421808 1.125451) (layer "B.Fab") (width 0.127))
-    (fp_arc (start -0.576537 0.906071) (mid -0.449563 0.779106) (end -0.322588 0.906071) (layer "B.Fab") (width 0.127))
+    (fp_arc (start -0.576537 0.906071) (mid -0.449562 0.77911) (end -0.322588 0.906071) (layer "B.Fab") (width 0.127))
     (fp_arc (start -0.724999 1.446) (mid -0.778512 1.423533) (end -0.800692 1.369901) (layer "B.Fab") (width 0.127))
     (fp_arc (start -0.800692 -1.398928) (mid -0.778507 -1.452548) (end -0.724999 -1.475002) (layer "B.Fab") (width 0.127))
@@
   )
   (footprint "Resistor_SMD:R_0603_1608Metric" (layer "B.Cu")
-    (at 27.051 -17.907 90)
+    (at 26.797 -17.907 90)
     (descr "Resistor SMD 0603 (1608 Metric), square (rectangular) end terminal, IPC_7351 nominal, (Body size source: IPC-SM-782 page 72, https://www.pcb-3d.com/wordpress/wp-content/uploads/ipc-sm-782a_amendment_1_and_2.pdf), generated with kicad-footprint-generator")
     (tags "resistor")
@@
       (effects (font (size 1 1) (thickness 0.15)) (justify mirror))
     )
-    (fp_text user "*" (at -1.27 1.27 90 unlocked) (layer "B.SilkS")
+    (fp_text user "*" (at -1.524 1.778 90 unlocked) (layer "B.SilkS")
       (effects (font (size 1 1) (thickness 0.15)) (justify mirror))
     )
